File: 2-Hardware/Kill_Board/ISU_LTA_Kill_Board.sch (KiCad schematic (older format))
At the start: 36 parts, among them P1 CONN_01X02, P10 CONN_2, P11 CONN_2, P12 CONN_2, P13 CONN_2, P14 CONN_2, P15 CONN_2, P16 CONN_2, P17 CONN_2, P18 CONN_2, P2 CONN_01X02, P3 CONN_01X02, P4 CONN_01X03, P5 CONN_01X03, P6 CONN_01X03, P7 CONN_2, P8 CONN_2, P9 CONN_2, Q1 NMOS+PMOS, Q2 N-CH, Q3 N-CH, U1 ADAFRUIT_FEATHER, U2 LM2937

Commit message: Updates to schematic
added current sense resistor, added buzzer.
Parts:
- removed P11, P13, P15, P17, P7, P9: CONN_2, Connectors:DEANS, symbol CONN_2
- added BZ?: Buzzer, symbol Device:Buzzer
- added R?: R_Shunt_US, symbol Device:R_Shunt_US
- BT1: footprint Connectors:DEANS -> Wire_Pads:SolderWirePad_2x_1-5mmDrill; symbol BATTERY -> ISU_LTA_Kill_Board-rescue:BATTERY
- C1, C2: symbol C-RESCUE-ISU_LTA_Kill_Board -> ISU_LTA_Kill_Board-rescue:C-RESCUE-ISU_LTA_Kill_Board
- D1: symbol LED-RESCUE-ISU_LTA_Kill_Board -> ISU_LTA_Kill_Board-rescue:LED-RESCUE-ISU_LTA_Kill_Board
- P1, P2, P3: symbol CONN_01X02 -> ISU_LTA_Kill_Board-rescue:CONN_01X02
- P10, P12, P14, P16, P18, P8: symbol CONN_2 -> ISU_LTA_Kill_Board-rescue:CONN_2
- P4, P5, P6: symbol CONN_01X03 -> ISU_LTA_Kill_Board-rescue:CONN_01X03
- Q1: symbol NMOS+PMOS -> ISU_LTA_Kill_Board-rescue:NMOS+PMOS
- Q2, Q3: symbol MOS_3-Term -> ISU_LTA_Kill_Board-rescue:MOS_3-Term
- R1: value 649k -> 75K; symbol R-RESCUE-ISU_LTA_Kill_Board -> ISU_LTA_Kill_Board-rescue:R-RESCUE-ISU_LTA_Kill_Board
- R2: value 330k -> 33k; symbol R-RESCUE-ISU_LTA_Kill_Board -> ISU_LTA_Kill_Board-rescue:R-RESCUE-ISU_LTA_Kill_Board
- R3, R4, R5, R6, R7, R8: symbol R-RESCUE-ISU_LTA_Kill_Board -> ISU_LTA_Kill_Board-rescue:R-RESCUE-ISU_LTA_Kill_Board
- S1: symbol DPDT -> ISU_LTA_Kill_Board-rescue:DPDT
- U1: symbol ADAFRUIT_FEATHER -> ISU_LTA_Kill_Board-rescue:ADAFRUIT_FEATHER
- U2: symbol LM2937 -> ISU_LTA_Kill_Board-rescue:LM2937
Connections:
- wire segments 96 -> 118
Other:
- note removed: "Deans Connectors"
- note removed: "Micro Deans Connectors"

Commit message: Fixed some issues with the schedmatic
Parts:
- removed BZ?: Buzzer, symbol Device:Buzzer
Changed lines of the file:
@@
 Sheet 1 1
 Title "ISU LTA Remote-Off & Telemetry System"
-Date "2018-07-24"
+Date "2018-10-30"
 Rev "E"
 Comp "Iowa State University"
@@
 Text Label 4600 4600 2    60   ~ 0
 Ctrl
-Text Label 1500 1400 2    60   ~ 0
-V_Sense
 Text Label 2750 4600 2    60   ~ 0
 V_Sense
@@
 Connection ~ 3100 4000
 Wire Wire Line
-	1500 1400 1900 1400
-Wire Wire Line
 	3500 2400 4400 2400
 Wire Wire Line
@@
 	10200 3600 10200 6050
 $Comp
-L Device:Buzzer BZ?
-U 1 1 5B5E43C3
-P 6850 2350
-F 0 "BZ?" H 7003 2379 50  0000 L CNN
-F 1 "Buzzer" H 7003 2288 50  0000 L CNN
-F 2 "" V 6825 2450 50  0001 C CNN
-F 3 "~" V 6825 2450 50  0001 C CNN
-	1    6850 2350
-	1    0    0    -1
-$EndComp
-$Comp
 L Device:R_Shunt_US R?
 U 1 1 5B5E680A
@@
 Wire Wire Line
 	2000 3600 2000 4300
+Wire Wire Line
+	3500 2100 4350 2100
+Text Label 4300 2100 0    50   ~ 0
+V_Sense
 $EndSCHEMATC
