File: 2-Hardware/Kill_Board/ISU_LTA_Kill_Board.kicad_sch (KiCad schematic)
At the start: 40 parts, among them P1 CONN_01X02, P10 CONN_2, P11 CONN_2, P12 CONN_2, P13 CONN_2, P2 CONN_01X02, P3 CONN_01X02, P4 CONN_01X03, P5 CONN_01X03, P6 CONN_01X03, P7 CONN_2, P8 CONN_2, Q1 NMOS+PMOS, Q2 N-CH, Q3 N-CH, Q4 FDN359AN mfet, U1 ADAFRUIT_FEATHER, U2 LM2937, U3 AZ1117-5.0, U4 NTS0104, U5 AZ1117-5.0

Commit message: New Revision
Parts:
- removed BEC1, P4, P5, P6: CONN_01X03, Pin_Headers:Pin_Header_Angled_1x03_Pitch2.54mm, symbol ISU_LTA_Kill_Board-rescue:CONN_01X03
- removed C1, C5: 0.1uF, Capacitors_SMD:C_0805_HandSoldering, symbol ISU_LTA_Kill_Board-rescue:C-RESCUE-ISU_LTA_Kill_Board
- removed C2, C6: 10uF, Capacitors_SMD:C_0805_HandSoldering, symbol ISU_LTA_Kill_Board-rescue:C-RESCUE-ISU_LTA_Kill_Board
- removed P1, P2, P3: CONN_01X02, Pin_Headers:Pin_Header_Angled_1x02_Pitch2.54mm, symbol ISU_LTA_Kill_Board-rescue:CONN_01X02
- removed Q4: FDN359AN mfet, TO_SOT_Packages_SMD:SOT-23, symbol ISU_LTA_Kill_Board:mosfet
- removed R9: 2k, Resistors_SMD:R_0805_HandSoldering, symbol ISU_LTA_Kill_Board-rescue:R-RESCUE-ISU_LTA_Kill_Board
- removed S1: DPDT, Buttons_Switches_ThroughHole:SW_CuK_JS202011CQN_DPDT_Straight, symbol ISU_LTA_Kill_Board-rescue:DPDT
- removed U1: ADAFRUIT_FEATHER, Adafruit:AdafruitFeather, symbol ISU_LTA_Kill_Board-rescue:ADAFRUIT_FEATHER
- removed U2: LM2937, TO_SOT_Packages_SMD:SOT-223, symbol ISU_LTA_Kill_Board-rescue:LM2937
- removed U3, U5: AZ1117-5.0, TO_SOT_Packages_SMD:SOT-223-3_TabPin2, symbol Regulator_Linear:AZ1117-5.0
- removed U4: NTS0104, Housings_SSOP:TSSOP-14_4.4x5mm_Pitch0.65mm, symbol ISU_LTA_Kill_Board:NTS0104
- added A1: Adafruit_Feather_M0_RFM9x_LoRa_Radio, Module:Adafruit_Feather_M0_RFM, symbol MCU_Module:Adafruit_Feather_M0_RFM9x_LoRa_Radio
- added D1: LED, LED_SMD:LED_0805_2012Metric_Pad1.15x1.40mm_HandSolder, symbol Device:LED
- added JP1: Jumper_2_Open, TestPoint:TestPoint_Bridge_Pitch2.54mm_Drill1.3mm, symbol Jumper:Jumper_2_Open
- added R3: 330, Resistor_SMD:R_0805_2012Metric_Pad1.20x1.40mm_HandSolder, symbol Device:R_US
- added SW1: SW_SPDT, LED_SMD:LED_0805_2012Metric_Pad1.15x1.40mm_HandSolder, symbol Switch:SW_SPDT
- added U1: LM1084-5.0, Package_TO_SOT_THT:TO-220-3_Horizontal_TabDown, symbol Regulator_Linear:LM1084-5.0
- C1: renamed from C3; value 0.1uF -> 1uF
- renumbered C4 to C2, D1 to D2, P7 to P1, P8 to P2, P10 to P3, P11 to P4, P12 to P5, P13 to P6, R3 to R4, R4 to R5, R5 to R6, R6 to R7, R7 to R8, R8 to R9
Connections:
- net +5V: now also JP1.2 (B), U1.2 (VO)
- net +BATT: now also R1.1
- net Ctrl: now also A1.7 (A2)
- net GND: now also A1.4 (GND), D1.1 (K), SW1.1 (A), U1.1 (GND)
- net V_Sense: now also A1.6 (A1)
- net at C1.1: now also U1.3 (VI); no longer R1.1
- net at R7.1, R8.1: now also SW1.2 (B)
- net at Q1.4 (S), Q1.6 (D): now also SW1.3 (C)
- new net: D1.2 (A), R3.1
- new net: A1.19 (D5), R3.2
- new net: A1.26 (USB), JP1.1 (A)
- no-connect marks 1 -> 0
Other:
- moved on the sheet: C1, C2, R1, R2

Commit message: Added IR stuff
Parts:
- added J? (x2): Conn_01x03_Male, symbol Connector:Conn_01x03_Male
- added U? (x2): TSOP382xx, OptoDevice:Vishay_MINICAST-3Pin, symbol Interface_Optical:TSOP382xx
Connections:
- net +5V: now also J?.2 (Pin_2), J?.2 (Pin_2), U?.3 (Vs), U?.3 (Vs)
- net GND: now also U?.2 (GND), U?.2 (GND)
- net at A1.20 (D6): now also U?.1 (OUT)
- net at A1.21 (D9): now also U?.1 (OUT)
